File: NeoRAMremix.kicad_pcb (KiCad board)
At the start: 2 copper layers, 58.2 x 84.1 mm, 28 parts, among them P1 C64-Exp-Port, Q1 2N3904, SW1 Reset, U1 HM628512BFP-5, U2 HM628512BFP-5, U3 HM628512BFP-5, U4 HM628512BFP-5

Commit message: Fixed footprint.
Other:
- board text added: "2019 Rev.2"
- board text removed: "2019 Rev.1"
